Commit message: link: dashboard + 3D URDF viewer with cached CAD assets
- Import OneDrive Rudy CAD library under `cad/` (LFS-tracked SLDPRT/STEP/STL/3MF/PDF/PNG); excludes MotorStudio vendor binaries.
- Convert curated STLs to glb under `ros/src/description/meshes/`; reference real meshes from `robot.urdf.xacro` via a new `mesh_link` macro.
- New `link/scripts/bake-urdf.mjs` runs xacro (with checked-in fallback), copies meshes, rewrites package URIs, and emits `manifest.json` (sha256 + size + mtime per asset).
- New `link/src/lib/asset-cache.ts`: IndexedDB-backed, hash-invalidated cache for the URDF + meshes; viewer + dashboard preview load through it.
- New rudydae endpoints: `GET /api/system` (Pi metrics with mock fallback) and `/api/reminders` CRUD (file-backed, audit-logged); ts-rs types regenerated.
- Replace `/` redirect with an Overview dashboard composing system-health, actuator-status, reminders, robot-preview, connection, and cache-status cards.
- Replace `/viz` ComingSoon with the live `UrdfViewer` + controls; add Overview entry to the app shell nav.

Made-with: Cursor

File: ros/src/description/urdf/robot.urdf.xacro (robot description, xacro)
@@ -46,4 +46,31 @@
     </link>
   </xacro:macro>
+  <!--
+    mesh_link: real glTF mesh as visual, conservative box as collision +
+    inertial. Use for printed/machined parts whose silhouette matters in
+    the operator console. Mesh meters; collision box dimensions are
+    bounding-box approximations (kept cheap for any future physics pass).
+    Source meshes regenerate via scripts/convert-meshes-to-glb.mjs.
+  -->
+  <xacro:macro name="mesh_link" params="name mesh sx sy sz rgba mass mesh_xyz:='0 0 0' mesh_rpy:='0 0 0' mesh_scale:='1 1 1'">
+    <link name="${name}">
+      <visual>
+        <origin xyz="${mesh_xyz}" rpy="${mesh_rpy}"/>
+        <geometry>
+          <mesh filename="package://description/meshes/${mesh}" scale="${mesh_scale}"/>
+        </geometry>
+        <material name="${name}_mat">
+          <color rgba="${rgba}"/>
+        </material>
+      </visual>
+      <collision>
+        <origin xyz="0 0 0" rpy="0 0 0"/>
+        <geometry>
+          <box size="${sx} ${sy} ${sz}"/>
+        </geometry>
+      </collision>
+      <xacro:box_inertial m="${mass}" x="${sx}" y="${sy}" z="${sz}"/>
+    </link>
+  </xacro:macro>
   <!-- Macro: revolute joint with hard limits, dynamics, soft safety band (~0.12 rad inside hard stops) -->
   <xacro:macro name="robot_revolute" params="name parent child axis lower upper soft_lower soft_upper origin_xyz origin_rpy">
@@ -84,7 +111,14 @@
     origin_xyz="0 0 0.23"
     origin_rpy="0 0 0"/>
-  <!-- Left arm links (visual/collision only; joint origins define kinematics) -->
-  <xacro:box_link name="l_shoulder_pitch_link" sx="0.08" sy="0.08" sz="0.14" rgba="0.2 0.55 0.3 1" mass="0.6"/>
-  <xacro:box_link name="l_shoulder_roll_link" sx="0.10" sy="0.10" sz="0.12" rgba="0.2 0.55 0.3 1" mass="0.5"/>
+  <!--
+    Left arm links. Joint origins define kinematics; visual geometry is the
+    shoulder housing mesh where available, primitive boxes elsewhere.
+  -->
+  <xacro:mesh_link name="l_shoulder_pitch_link"
+    mesh="shoulder_housing.glb"
+    sx="0.08" sy="0.08" sz="0.14" rgba="0.2 0.55 0.3 1" mass="0.6"/>
+  <xacro:mesh_link name="l_shoulder_roll_link"
+    mesh="shoulder_housing_cap.glb"
+    sx="0.10" sy="0.10" sz="0.12" rgba="0.2 0.55 0.3 1" mass="0.5"/>
   <xacro:box_link name="l_upper_arm_link" sx="0.09" sy="0.09" sz="0.22" rgba="0.2 0.55 0.3 1" mass="0.7"/>
   <xacro:box_link name="l_forearm_link" sx="0.08" sy="0.08" sz="0.20" rgba="0.15 0.45 0.25 1" mass="0.5"/>
@@ -134,7 +168,13 @@
     origin_xyz="0 0 -0.18"
     origin_rpy="0 0 0"/>
-  <!-- Right arm -->
-  <xacro:box_link name="r_shoulder_pitch_link" sx="0.08" sy="0.08" sz="0.14" rgba="0.25 0.35 0.65 1" mass="0.6"/>
-  <xacro:box_link name="r_shoulder_roll_link" sx="0.10" sy="0.10" sz="0.12" rgba="0.25 0.35 0.65 1" mass="0.5"/>
+  <!-- Right arm: mirror of left, with the shoulder housing rotated 180 deg about Z. -->
+  <xacro:mesh_link name="r_shoulder_pitch_link"
+    mesh="shoulder_housing.glb"
+    mesh_rpy="0 0 3.14159"
+    sx="0.08" sy="0.08" sz="0.14" rgba="0.25 0.35 0.65 1" mass="0.6"/>
+  <xacro:mesh_link name="r_shoulder_roll_link"
+    mesh="shoulder_housing_cap.glb"
+    mesh_rpy="0 0 3.14159"
+    sx="0.10" sy="0.10" sz="0.12" rgba="0.25 0.35 0.65 1" mass="0.5"/>
   <xacro:box_link name="r_upper_arm_link" sx="0.09" sy="0.09" sz="0.22" rgba="0.25 0.35 0.65 1" mass="0.7"/>
   <xacro:box_link name="r_forearm_link" sx="0.08" sy="0.08" sz="0.20" rgba="0.2 0.3 0.55 1" mass="0.5"/>

Commit message: feat(ros): add arm-tip MoveIt scaffold
Add sim-first right-arm-tip planning around the 5-DOF arm
before wiring hardware execution through cortex.

File: ros/src/description/urdf/robot.urdf.xacro (robot description, xacro)
@@ -2,5 +2,7 @@
 <!--
   Rudy humanoid — kinematic skeleton for Phase 1.
-  Joint limits mirror mr_robot config/robot.yaml (RS03 caps: 60 Nm, 50 rad/s).
+  Arm model targets 5 DOF per side: shoulder pitch/roll, upper-arm yaw,
+  elbow pitch, lower-arm yaw. Joint limits mirror mr_robot config/robot.yaml
+  where available (RS03 caps: 60 Nm, 50 rad/s).
   Frame convention: x forward, y left, z up. Left arm attaches on +y side of torso.
 -->
@@ -123,4 +125,6 @@
   <xacro:box_link name="l_upper_arm_link" sx="0.09" sy="0.09" sz="0.22" rgba="0.2 0.55 0.3 1" mass="0.7"/>
   <xacro:box_link name="l_forearm_link" sx="0.08" sy="0.08" sz="0.20" rgba="0.15 0.45 0.25 1" mass="0.5"/>
+  <xacro:box_link name="l_lower_arm_yaw_link" sx="0.07" sy="0.07" sz="0.07" rgba="0.15 0.45 0.25 1" mass="0.35"/>
+  <xacro:box_link name="l_arm_tip" sx="0.05" sy="0.05" sz="0.05" rgba="0.1 0.35 0.2 1" mass="0.15"/>
   <!-- arm_left from robot.yaml -->
   <xacro:robot_revolute
@@ -168,4 +172,20 @@
     origin_xyz="0 0 -0.18"
     origin_rpy="0 0 0"/>
+  <xacro:robot_revolute
+    name="l_lower_arm_yaw_joint"
+    parent="l_forearm_link"
+    child="l_lower_arm_yaw_link"
+    axis="0 0 1"
+    lower="-1.57"
+    upper="1.57"
+    soft_lower="-1.45"
+    soft_upper="1.45"
+    origin_xyz="0 0 -0.14"
+    origin_rpy="0 0 0"/>
+  <joint name="l_lower_arm_yaw_to_tip" type="fixed">
+    <origin xyz="0 0 -0.08" rpy="0 0 0"/>
+    <parent link="l_lower_arm_yaw_link"/>
+    <child link="l_arm_tip"/>
+  </joint>
   <!-- Right arm: mirror of left, with the shoulder housing rotated 180 deg about Z. -->
   <xacro:mesh_link name="r_shoulder_pitch_link"
@@ -179,4 +199,6 @@
   <xacro:box_link name="r_upper_arm_link" sx="0.09" sy="0.09" sz="0.22" rgba="0.25 0.35 0.65 1" mass="0.7"/>
   <xacro:box_link name="r_forearm_link" sx="0.08" sy="0.08" sz="0.20" rgba="0.2 0.3 0.55 1" mass="0.5"/>
+  <xacro:box_link name="r_lower_arm_yaw_link" sx="0.07" sy="0.07" sz="0.07" rgba="0.2 0.3 0.55 1" mass="0.35"/>
+  <xacro:box_link name="r_arm_tip" sx="0.05" sy="0.05" sz="0.05" rgba="0.15 0.25 0.45 1" mass="0.15"/>
   <xacro:robot_revolute
     name="r_shoulder_pitch_joint"
@@ -223,3 +245,74 @@
     origin_xyz="0 0 -0.18"
     origin_rpy="0 0 0"/>
+  <xacro:robot_revolute
+    name="r_lower_arm_yaw_joint"
+    parent="r_forearm_link"
+    child="r_lower_arm_yaw_link"
+    axis="0 0 1"
+    lower="-1.57"
+    upper="1.57"
+    soft_lower="-1.45"
+    soft_upper="1.45"
+    origin_xyz="0 0 -0.14"
+    origin_rpy="0 0 0"/>
+  <joint name="r_lower_arm_yaw_to_tip" type="fixed">
+    <origin xyz="0 0 -0.08" rpy="0 0 0"/>
+    <parent link="r_lower_arm_yaw_link"/>
+    <child link="r_arm_tip"/>
+  </joint>
+  <ros2_control name="RudySystem" type="system">
+    <hardware>
+      <plugin>control/TopicLoopbackHardware</plugin>
+    </hardware>
+    <joint name="l_shoulder_pitch_joint">
+      <command_interface name="position"/>
+      <state_interface name="position"/>
+      <state_interface name="velocity"/>
+    </joint>
+    <joint name="l_shoulder_roll_joint">
+      <command_interface name="position"/>
+      <state_interface name="position"/>
+      <state_interface name="velocity"/>
+    </joint>
+    <joint name="l_upper_arm_yaw_joint">
+      <command_interface name="position"/>
+      <state_interface name="position"/>
+      <state_interface name="velocity"/>
+    </joint>
+    <joint name="l_elbow_pitch_joint">
+      <command_interface name="position"/>
+      <state_interface name="position"/>
+      <state_interface name="velocity"/>
+    </joint>
+    <joint name="l_lower_arm_yaw_joint">
+      <command_interface name="position"/>
+      <state_interface name="position"/>
+      <state_interface name="velocity"/>
+    </joint>
+    <joint name="r_shoulder_pitch_joint">
+      <command_interface name="position"/>
+      <state_interface name="position"/>
+      <state_interface name="velocity"/>
+    </joint>
+    <joint name="r_shoulder_roll_joint">
+      <command_interface name="position"/>
+      <state_interface name="position"/>
+      <state_interface name="velocity"/>
+    </joint>
+    <joint name="r_upper_arm_yaw_joint">
+      <command_interface name="position"/>
+      <state_interface name="position"/>
+      <state_interface name="velocity"/>
+    </joint>
+    <joint name="r_elbow_pitch_joint">
+      <command_interface name="position"/>
+      <state_interface name="position"/>
+      <state_interface name="velocity"/>
+    </joint>
+    <joint name="r_lower_arm_yaw_joint">
+      <command_interface name="position"/>
+      <state_interface name="position"/>
+      <state_interface name="velocity"/>
+    </joint>
+  </ros2_control>
 </robot>
